File: fristracker/fristracker.kicad_sch (KiCad schematic)
At the start: 15 parts, among them J1 SMA_Edge_SMD, P1 Conn_USB_A_Plain, SW1 Switch_Tactile_Omron, U1 ESP32-PICO-V3-02, U2 NEO-6M, U3 CH340E, U4 TLV75733PDRV, U5 NRF24L01+PA+LNA

Commit message: FInal commit?
Parts:
- C1: footprint PCM_SparkFun-Semiconductor-Standard:WDFN-6_2x2mm -> PCM_Capacitor_THT_US_AKL:C_Disc_D5.0mm_W2.5mm_P5.00mm
- C3: footprint PCM_Capacitor_THT_AKL:C_Disc_D4.3mm_W1.9mm_P5.00mm -> PCM_Capacitor_THT_AKL:CP_Radial_Tantal_D5.0mm_P5.00mm
- R1, R2: footprint PCM_Resistor_THT_AKL:R_Axial_DIN0411_L9.9mm_D3.6mm_P15.24mm_Horizontal -> PCM_Resistor_SMD_AKL:R_0603_1608Metric
Changed lines of the file:
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@@
+	)
+	(junction
+		(at 82.55 41.91)
+		(diameter 0)
+		(color 0 0 0 0)
 	)
 	(junction
@@
 	)
 	(junction
-		(at 82.55 40.64)
-		(diameter 0)
-		(color 0 0 0 0)
-	)
-	(junction
 		(at 82.55 50.8)
 		(diameter 0)
@@
 	(wire
 		(pts
-			(xy 82.55 40.64) (xy 82.55 50.8)
-		)
-		(stroke
-			(width 0)
-			(type default)
-		)
-	)
-	(wire
-		(pts
 			(xy 26.67 86.36) (xy 26.67 58.42)
 		)
@@
 	(wire
 		(pts
-			(xy 82.55 40.64) (xy 66.04 40.64)
-		)
-		(stroke
-			(width 0)
-			(type default)
-		)
-	)
-	(wire
-		(pts
 			(xy 227.33 25.4) (xy 237.49 25.4)
 		)
@@
 	(wire
 		(pts
+			(xy 66.04 41.91) (xy 82.55 41.91)
+		)
+		(stroke
+			(width 0)
+			(type default)
+		)
+	)
+	(wire
+		(pts
 			(xy 30.48 81.28) (xy 30.48 74.93)
 		)
@@
 	(wire
 		(pts
+			(xy 82.55 41.91) (xy 82.55 50.8)
+		)
+		(stroke
+			(width 0)
+			(type default)
+		)
+	)
+	(wire
+		(pts
 			(xy 38.1 43.18) (xy 48.26 43.18)
 		)
@@
 	(wire
 		(pts
-			(xy 82.55 13.97) (xy 82.55 40.64)
+			(xy 82.55 13.97) (xy 82.55 41.91)
 		)
 		(stroke
@@
 			)
 		)
-		(property "Footprint" "PCM_Resistor_THT_AKL:R_Axial_DIN0411_L9.9mm_D3.6mm_P15.24mm_Horizontal"
+		(property "Footprint" "PCM_Resistor_SMD_AKL:R_0603_1608Metric"
 			(at 112.522 86.36 0)
 			(hide yes)
@@
 			)
 		)
-		(property "Footprint" "PCM_Capacitor_THT_AKL:C_Disc_D4.3mm_W1.9mm_P5.00mm"
+		(property "Footprint" "PCM_Capacitor_THT_AKL:CP_Radial_Tantal_D5.0mm_P5.00mm"
 			(at 199.39 85.09 0)
 			(hide yes)
@@
 			)
 		)
-		(property "Footprint" "PCM_SparkFun-Semiconductor-Standard:WDFN-6_2x2mm"
+		(property "Footprint" "PCM_Capacitor_THT_US_AKL:C_Disc_D5.0mm_W2.5mm_P5.00mm"
 			(at 48.26 48.26 0)
 			(hide yes)
@@
 			)
 		)
-		(property "Footprint" "PCM_Resistor_THT_AKL:R_Axial_DIN0411_L9.9mm_D3.6mm_P15.24mm_Horizontal"
+		(property "Footprint" "PCM_Resistor_SMD_AKL:R_0603_1608Metric"
 			(at 71.882 91.44 0)
 			(hide yes)
