File: fristracker/fristracker.kicad_pcb (KiCad board)
At the start: 2 copper layers, 62.8 x 72.4 mm, 15 parts, among them J1 SMA_Edge_SMD, P1 Conn_USB_A_Plain, SW1 Switch_Tactile_Omron, U1 ESP32-PICO-V3-02, U2 NEO-6M, U3 CH340E, U4 TLV75733PDRV, U5 NRF24L01+PA+LNA

Commit message: FInal commit?
Parts:
- C1: footprint PCM_SparkFun-Semiconductor-Standard:WDFN-6_2x2mm -> PCM_Capacitor_THT_US_AKL:C_Disc_D5.0mm_W2.5mm_P5.00mm
- C3: footprint PCM_Capacitor_THT_AKL:C_Disc_D4.3mm_W1.9mm_P5.00mm -> PCM_Capacitor_THT_AKL:CP_Radial_Tantal_D5.0mm_P5.00mm
- R1, R2: footprint PCM_Resistor_THT_AKL:R_Axial_DIN0411_L9.9mm_D3.6mm_P15.24mm_Horizontal -> PCM_Resistor_SMD_AKL:R_0603_1608Metric
- moved C2 7.59 mm to (121.5, 88.5)
- moved R2 4.64 mm to (114.0, 106.5), turned to -90 degrees
- moved C1 2.51 mm to (113.0, 77.0)
- moved R1 2.33 mm to (121.5, 129.0)
- moved C3 0.16 mm to (130.0, 73.0)
Routing:
- net Net-(C2-+): track 108.9 -> 149.3 mm, vias 3 -> 7
- net Net-(C4-+): track 39.5 -> 67.4 mm
- net GND: track 290.8 -> 285.0 mm, vias 10 -> 12
- net Net-(U1-IOA0): track 119.0 -> 115.8 mm
- net Net-(C1-+): track 27.9 -> 25.5 mm
Other:
- outline, holes or cut-outs redrawn

Commit message: Added personal Touch!
Routing:
- net Net-(J1-In): track 13.8 -> 11.9 mm
Other:
- board text added: "Made by Jakob @ Hackclub Halflive"
Changed lines of the file:
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@@
 		(layer "Edge.Cuts")
+	)
+	(gr_text "Made by \nJakob @\nHackclub \nHalflive"
+		(at 147 88.5 0)
+		(layer "Edge.Cuts")
+		(effects
+			(font
+				(size 1 1)
+				(thickness 0.15)
+			)
+			(justify left bottom)
+		)
 	)
 	(segment
@@
 	)
 	(segment
-		(start 109.05 103.65)
-		(end 108.25 102.85)
+		(start 108.85 102.85)
+		(end 106.05 102.85)
 		(width 0.8)
 		(layer "F.Cu")
@@
 	)
 	(segment
-		(start 107.05 105.65)
-		(end 109.05 103.65)
+		(start 109 110.6)
+		(end 109 103)
+		(width 0.8)
+		(layer "F.Cu")
+		(net "Net-(J1-In)")
+	)
+	(segment
+		(start 109 103)
+		(end 108.85 102.85)
+		(width 0.8)
+		(layer "F.Cu")
+		(net "Net-(J1-In)")
+	)
+	(segment
+		(start 109.05 110.65)
+		(end 109 110.6)
 		(width 0.8)
 		(layer "F.Cu")
@@
 		(start 109.05 111.9)
 		(end 109.05 110.65)
-		(width 0.8)
-		(layer "F.Cu")
-		(net "Net-(J1-In)")
-	)
-	(segment
-		(start 107.05 109.65)
-		(end 107.05 105.65)
-		(width 0.8)
-		(layer "F.Cu")
-		(net "Net-(J1-In)")
-	)
-	(segment
-		(start 108.25 102.85)
-		(end 106.05 102.85)
-		(width 0.8)
-		(layer "F.Cu")
-		(net "Net-(J1-In)")
-	)
-	(segment
-		(start 108.05 109.65)
-		(end 107.05 109.65)
-		(width 0.8)
-		(layer "F.Cu")
-		(net "Net-(J1-In)")
-	)
-	(segment
-		(start 109.05 110.65)
-		(end 108.05 109.65)
 		(width 0.8)
 		(layer "F.Cu")
@@
 		(polygon
 			(pts
-				(xy 154 84.5) (xy 159 96.5) (xy 159.5 104.999998) (xy 153.499999 120.000001) (xy 146 127.5) (xy 136 132)
-				(xy 123.5 132.5) (xy 119.33 131.5) (xy 115 129.85) (xy 108.5 125.5) (xy 100 114) (xy 97.95 106)
-				(xy 97.95 96.5) (xy 101.5 86) (xy 110.5 76.5) (xy 121 72) (xy 134.5 71.5) (xy 141 74) (xy 150 79.5)
+				(xy 157.102855 89.859993) (xy 159 96.5) (xy 159.5 104.999998) (xy 153.499999 120.000001) (xy 146 127.5)
+				(xy 136 132) (xy 123.5 132.5) (xy 119.33 131.5) (xy 115 129.85) (xy 108.5 125.5) (xy 100 114) (xy 97.95 106)
+				(xy 97.95 96.5) (xy 101.5 86) (xy 110.5 76.5) (xy 121 72) (xy 134.5 71.5) (xy 145.55 75.95) (xy 147.5 88.5)
 			)
 		)
