File: fristracker/fristracker_RCF/fristracker_RCF.kicad_pcb (KiCad board)
At the start: 2 copper layers, 15.5 x 98 mm, 12 parts, among them P1 Conn_USB_A_Plain, SW1 Switch_Tactile_Omron, U1 ESP32-PICO-V3-02, U3 CH340E, U4 TLV75733PDRV, U5 NRF24L01+PA+LNA

Commit message: Added personal Touch!
Other:
- board text added: "Made by Jakob @ Hackclub Halflive"
